Commit message: Add MoveIt2 integration, Servo config, and Gazebo simulation improvements
- Add MoveIt Servo configuration and launch files for joystick IK control
- Add combined Gazebo + MoveIt Servo launch (falcon_arm_servo_sim.launch.py)
- Update URDF with Gazebo PD gains and fix mock hardware calculate_dynamics issue
- Refactor Gazebo launch and update controller configs
- Add CLAUDE.md with project documentation
- Remove unused display and ros2_control launch files

Co-Authored-By: Claude Opus 4.6 <noreply@anthropic.com>

File: src/falcon_robotic_arm_description/urdf/falcon_robotic_arm.ros2control.xacro (robot description, xacro)
@@ -24,12 +24,4 @@
   *  Co-Author:      RON NIRVIN J
   *
-  *  FIX (2026-03-15):
-  *    Added explicit xacro:arg declarations for sim_gazebo, hardware_type, serial_port
-  *    so this file can be safely evaluated standalone (e.g. by MoveIt Setup Assistant).
-  *    Replaced bare ${hardware_type == 'real'} expressions — which fail because
-  *    hardware_type is an arg, not a property — with a local xacro:property 'hw_type'
-  *    that is set from $(arg hardware_type).  The ${hw_type == 'real'} expression then
-  *    evaluates correctly in both standalone and included contexts.
-  *
   *  Usage:
   *    Included automatically by falcon_robotic_arm.xacro — do not include directly.
@@ -37,12 +29,5 @@
 -->
 <robot xmlns:xacro="http://www.ros.org/wiki/xacro">
-  <!-- Declare args here so xacro can resolve them when this file is processed
-       both standalone (MoveIt Setup Assistant) and as an include. -->
-  <xacro:arg name="sim_gazebo"    default="false"/>
-  <xacro:arg name="hardware_type" default="fake"/>
-  <xacro:arg name="serial_port"   default="/dev/ttyACM0"/>
-  <!-- Resolve the arg into a property so it can be used in Python expressions
-       inside xacro:if / xacro:unless value="${...}" blocks. -->
-  <xacro:property name="hw_type" value="$(arg hardware_type)"/>
+  <xacro:property name="hardware_type" value="$(arg hardware_type)"/>
   <xacro:if value="$(arg sim_gazebo)">
     <ros2_control name="FalconArm" type="system">
@@ -136,8 +121,5 @@
   <xacro:unless value="$(arg sim_gazebo)">
     <ros2_control name="FalconArm" type="system">
-      <!-- FIX: was ${hardware_type == 'real'} — hardware_type is an xacro:arg, not a
-           property, so it cannot be used directly inside ${} Python expressions.
-           Use the hw_type property declared above instead. -->
-      <xacro:if value="${hw_type == 'real'}">
+      <xacro:if value="${hardware_type == 'real'}">
         <hardware>
           <plugin>falcon_arm_hardware/FalconArmHardwareInterface</plugin>
@@ -147,8 +129,7 @@
         </hardware>
       </xacro:if>
-      <xacro:unless value="${hw_type == 'real'}">
+      <xacro:unless value="${hardware_type == 'real'}">
         <hardware>
           <plugin>mock_components/GenericSystem</plugin>
-          <!--<param name="calculate_dynamics">true</param> -->
         </hardware>
       </xacro:unless>

File: src/falcon_robotic_arm_description/urdf/falcon_robotic_arm.xacro (robot description, xacro)
@@ -40,10 +40,9 @@
   <xacro:include filename="$(find falcon_robotic_arm_description)/urdf/falcon_robotic_arm.gazebo"/>
   <link name="world"/>
-  <!-- AFTER -->
-<joint name="world_fixed" type="fixed">
-  <origin xyz="0 0 0" rpy="-1.5708 0 0"/>
-  <parent link="world"/>
-  <child link="base_link"/>
-</joint>
+  <joint name="world_fixed" type="fixed">
+    <origin xyz="0 0 0" rpy="-1.5708 0 0"/>
+    <parent link="world"/>
+    <child link="base_link"/>
+  </joint>
   <link name="base_link">
     <inertial>

Commit message: Update joystick controls and unlock full joint rotation for MoveIt Servo
Remap gamepad: START=enable toggle, left stick=XY, right stick=Z+yaw,
LT/RT=gripper close/open, X=singularity recovery to safe "ready" pose.
Extend arm joint limits from ±90° to ±180° (full 360°) for flexibility
testing while keeping gripper limits unchanged (-0.7 to 0 rad).

Co-Authored-By: Claude Opus 4.6 <noreply@anthropic.com>

File: src/falcon_robotic_arm_description/urdf/falcon_robotic_arm.ros2control.xacro (robot description, xacro)
@@ -43,6 +43,6 @@
         <param name="position_proportional_gain">100.0</param>  <!-- vertical axis, negligible gravity -->
         <command_interface name="position">
-          <param name="min">-1.5708</param>
-          <param name="max">1.5708</param>
+          <param name="min">-3.14159</param>
+          <param name="max">3.14159</param>
         </command_interface>
         <state_interface name="position">
@@ -54,6 +54,6 @@
         <param name="position_proportional_gain">500.0</param>  <!-- shoulder: heaviest gravity load -->
         <command_interface name="position">
-          <param name="min">-1.5708</param>
-          <param name="max">1.5708</param>
+          <param name="min">-3.14159</param>
+          <param name="max">3.14159</param>
         </command_interface>
         <state_interface name="position">
@@ -65,6 +65,6 @@
         <param name="position_proportional_gain">300.0</param>  <!-- elbow: moderate gravity load -->
         <command_interface name="position">
-          <param name="min">-1.5708</param>
-          <param name="max">1.5708</param>
+          <param name="min">-3.14159</param>
+          <param name="max">3.14159</param>
         </command_interface>
         <state_interface name="position">
@@ -76,6 +76,6 @@
         <param name="position_proportional_gain">100.0</param>
         <command_interface name="position">
-          <param name="min">-1.5708</param>
-          <param name="max">1.5708</param>
+          <param name="min">-3.14159</param>
+          <param name="max">3.14159</param>
         </command_interface>
         <state_interface name="position">
@@ -87,6 +87,6 @@
         <param name="position_proportional_gain">100.0</param>
         <command_interface name="position">
-          <param name="min">-1.5708</param>
-          <param name="max">1.5708</param>
+          <param name="min">-3.14159</param>
+          <param name="max">3.14159</param>
         </command_interface>
         <state_interface name="position">
@@ -136,6 +136,6 @@
       <joint name="joint_1">
         <command_interface name="position">
-          <param name="min">-1.5708</param>
-          <param name="max">1.5708</param>
+          <param name="min">-3.14159</param>
+          <param name="max">3.14159</param>
         </command_interface>
         <state_interface name="position">
@@ -146,6 +146,6 @@
       <joint name="joint_2">
         <command_interface name="position">
-          <param name="min">-1.5708</param>
-          <param name="max">1.5708</param>
+          <param name="min">-3.14159</param>
+          <param name="max">3.14159</param>
         </command_interface>
         <state_interface name="position">
@@ -156,6 +156,6 @@
       <joint name="joint_3">
         <command_interface name="position">
-          <param name="min">-1.5708</param>
-          <param name="max">1.5708</param>
+          <param name="min">-3.14159</param>
+          <param name="max">3.14159</param>
         </command_interface>
         <state_interface name="position">
@@ -166,6 +166,6 @@
       <joint name="joint_4">
         <command_interface name="position">
-          <param name="min">-1.5708</param>
-          <param name="max">1.5708</param>
+          <param name="min">-3.14159</param>
+          <param name="max">3.14159</param>
         </command_interface>
         <state_interface name="position">
@@ -176,6 +176,6 @@
       <joint name="joint_5">
         <command_interface name="position">
-          <param name="min">-1.5708</param>
-          <param name="max">1.5708</param>
+          <param name="min">-3.14159</param>
+          <param name="max">3.14159</param>
         </command_interface>
         <state_interface name="position">

File: src/falcon_robotic_arm_description/urdf/falcon_robotic_arm.xacro (robot description, xacro)
@@ -218,5 +218,5 @@
     <child link="link_1" />
     <axis xyz="0 0 -1" />
-    <limit lower="-1.5708" upper="1.5708" effort="20" velocity="1" />
+    <limit lower="-3.14159" upper="3.14159" effort="20" velocity="1" />
   </joint>
   <joint name="joint_2" type="revolute">
@@ -225,5 +225,5 @@
     <child link="link_2" />
     <axis xyz="-0.0303599450227944 0 0.999539030622723" />
-    <limit lower="-1.5708" upper="1.5708" effort="50" velocity="1" />
+    <limit lower="-3.14159" upper="3.14159" effort="50" velocity="1" />
     <dynamics damping="0.5" friction="0.0"/>
   </joint>
@@ -233,5 +233,5 @@
     <child link="link_3" />
     <axis xyz="-0.0303599450227945 0 0.999539030622723" />
-    <limit lower="-1.5708" upper="1.5708" effort="30" velocity="1" />
+    <limit lower="-3.14159" upper="3.14159" effort="30" velocity="1" />
     <dynamics damping="0.3" friction="0.0"/>
   </joint>
@@ -241,5 +241,5 @@
     <child link="link_4" />
     <axis xyz="0.818727734388728 0.0296401954212068 0.573416389509484" />
-    <limit lower="-1.5708" upper="1.5708" effort="20" velocity="1" />
+    <limit lower="-3.14159" upper="3.14159" effort="20" velocity="1" />
   </joint>
   <joint name="joint_5" type="revolute">
@@ -248,5 +248,5 @@
     <child link="link_5" />
     <axis xyz="-0.0223564735183862 -0.233891765016945 -0.972005571151256" />
-    <limit lower="-1.5708" upper="1.5708" effort="20" velocity="1" />
+    <limit lower="-3.14159" upper="3.14159" effort="20" velocity="1" />
   </joint>
   <joint name="gripper_joint_1" type="revolute">
